Commit message: Add Gazebo World

File: description/robot_core.xacro (robot description, xacro)
@@ -21,5 +21,5 @@
         <parent link="base_link"/>
         <child link="chassis"/>
-        <origin xyz="0.1 0 0"/>
+        <origin xyz="-0.1 0 0"/>
     </joint>
     <link name="chassis">
@@ -41,4 +41,7 @@
         </xacro:inertial_box>
     </link>
+    <gazebo reference="chassis">
+        <material>Gazebo/White</material>
+    </gazebo>
     <!-- LEFT WHEEL Link-->
     <joint name="left_wheel_joint" type="continuous">
@@ -46,5 +49,5 @@
         <child link="left_wheel"/>
         <origin xyz="0 0.175 0" rpy="-${pi/2} 0 0"/>
-        <axes xyz="0 0 1"/>
+        <axis xyz="0 0 1"/>
     </joint>
     <link name="left_wheel">
@@ -64,4 +67,7 @@
         </xacro:inertial_cylinder>
     </link>
+    <gazebo reference="left_wheel">
+        <material>Gazebo/Blue</material>
+    </gazebo>
     <!-- RIGHT WHEEL Link-->
     <joint name="right_wheel_joint" type="continuous">
@@ -69,5 +75,5 @@
         <child link="right_wheel"/>
         <origin xyz="0 -0.175 0" rpy="${pi/2} 0 0"/>
-        <axes xyz="0 0 -1"/>
+        <axis xyz="0 0 -1"/>
     </joint>
     <link name="right_wheel">
@@ -87,9 +93,12 @@
         </xacro:inertial_cylinder>
     </link>
+    <gazebo reference="right_wheel">
+        <material>Gazebo/Blue</material>
+    </gazebo>
     <!-- CASTER WHEEL LINK-->
     <joint name="caster_wheel_joint" type="fixed">
         <parent link="chassis"/>
         <child link="wheel_caster"/>
-        <origin xyz="0 0.24 0"/>
+        <origin xyz="0.24 0 0"/>
     </joint>
     <link name="wheel_caster">
@@ -109,3 +118,8 @@
         </xacro:inertial_sphere>
     </link>
+    <gazebo reference="wheel_caster">
+        <material>Gazebo/Black</material>
+        <mu1 value="0.001"/>
+        <mu2 value="0.001"/>
+    </gazebo>
 </robot>
